Commit message: Fixed up urdfs

File: project/environment.urdf (robot description, URDF)
Before this commit: robot env, 3 links, 2 joints
Joints:
- joint place_ring: limit lower=-2.8973 upper=2.8973 effort=87 velocity=2.1750 -> lower=-3.14159265359 upper=3.14159265359 effort=100 velocity=3.14159265359; origin xyz=0.0 0.0 0.0 rpy=1.57079632679 0 0 -> xyz=0 0 0 rpy=1.57079632679 0 0
- joint place_stand: limit lower=-2.8973 upper=2.8973 effort=87 velocity=2.1750 -> lower=-3.14159265359 upper=3.14159265359 effort=100 velocity=3.14159265359; origin xyz=0.75 0.745 0 rpy=0 -1.57079632679 0 -> xyz=0 0 0 rpy=0 -1.57079632679 0

File: project/punching_bag.urdf (robot description, URDF)
Before this commit: robot punching_bag, 4 links, 3 joints
Links:
- link bag: geometry visual mesh filename=../../../model/boxing_ring/meshes/punchbag_blender.obj
- link link0: mass 0.1 -> 1e-16
- link link1: mass 0.1 -> 1e-16
- link link2: mass 3 -> 1e-16
Joints:
- joint joint1: origin xyz=0.75 0 0.7 rpy=1.57079632679 0 1.57079632679 -> xyz=0 0 0 rpy=0 0 0
- joint joint2: axis 0 0 1 -> 0 1 0
- joint joint3: axis 0 0 1 -> 1 0 0

File: project/toro.urdf (robot description, URDF)
Before this commit: robot DLR_TORO, 34 links, 33 joints
Joints:
- joint j13: origin (none) -> xyz=0 0 0 rpy=0 0 0
- joint j22: origin (none) -> xyz=0 0 0 rpy=0 0 0
- joint j3: origin (none) -> xyz=0 0 0 rpy=0 0 0
- joint j9: origin (none) -> xyz=0 0 0 rpy=0 0 0

Commit message: Rotated bag stand

File: project/environment.urdf (robot description, URDF)
Before this commit: robot env, 3 links, 2 joints
Joints:
- joint place_stand: origin xyz=0 0 0 rpy=0 -1.57079632679 0 -> xyz=0 0 0 rpy=0 3.14159265359 0
