Commit message: Added boxing ring, punching bag stand

File: project/punching_bag.urdf (robot description, URDF)
Before this commit: robot punching_bag, 4 links, 3 joints
Joints:
- joint joint1: origin xyz=0.75 0 0.9 rpy=1.57079632679 0 0 -> xyz=0.75 0 0.7 rpy=1.57079632679 0 1.57079632679

Commit message: Minor punching bag updates to prep for punching_bag controller

File: project/punching_bag.urdf (robot description, URDF)
Before this commit: robot punching_bag, 4 links, 3 joints
Links:
- link bag: geometry collision mesh filename=../../../model/boxing_ring/meshes/collision/punchbag_collis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; visual mesh filename=../../../model/boxing_ring/meshes/punchbag_blender.obj
Joints:
- joint joint1: limit lower=-2.8973 upper=2.8973 effort=87 velocity=2.1750 -> lower=-3.14159265359 upper=3.14159265359 effort=100 velocity=3.14159265359
- joint joint2: limit lower=-1.7628 upper=1.7628 effort=87 velocity=2.1750 -> lower=-3.14159265359 upper=3.14159265359 effort=100 velocity=3.14159265359
- joint joint3: limit lower=-2.8973 upper=2.8973 effort=87 velocity=2.1750 -> lower=-3.14159265359 upper=3.14159265359 effort=100 velocity=3.14159265359

Commit message: Position-only control as recommended by William

File: project/punching_bag.urdf (robot description, URDF)
Before this commit: robot punching_bag, 4 links, 3 joints
Links:
- link bag: geometry visual mesh filename=../../../model/boxing_ring/meshes/punchbag_blender.obj; visual sphere radius=0.3 rgba=0.5 0.5 1

Commit message: Added dodge to state machine and started defining dodge position

File: project/punching_bag.urdf (robot description, URDF)
Before this commit: robot punching_bag, 4 links, 3 joints
Links:
- link bag: geometry visual mesh filename=../../../model/boxing_ring/meshes/punchbag_blender.obj

Commit message: Collisions on. Fixed weird wrist joint. Attempted to increase gains while recovering. Sorry these aren't multiple commits.

File: project/punching_bag.urdf (robot description, URDF)
Before this commit: robot punching_bag, 4 links, 3 joints
Links:
- link bag: geometry collision cylinder length=0.8 radius=0.14; visual mesh filename=../../../model/boxing_ring/meshes/punchbag_blender.obj

File: project/toro.urdf (robot description, URDF)
Before this commit: robot DLR_TORO, 34 links, 33 joints
Links:
- link la_link6: geometry collision sphere radius=0.03; visual mesh filename=../../../model/toro/meshes/obj/wrist.stl.obj
- link ra_link6: geometry collision sphere radius=0.03; visual mesh filename=../../../model/toro/meshes/obj/wrist.stl.obj
Joints:
- joint j19: type revolute -> fixed
- joint j25: type revolute -> fixed
